Commit message: 12

File: patrol_bringup/urdf/patrol_robot.urdf (robot description, URDF)
Before this commit: robot patrol_robot, 6 links, 5 joints
Links:
- link ultrasonic_link: geometry visual cylinder length=0.03 radius=0.015

Commit message: 30

File: patrol_bringup/urdf/patrol_robot.urdf (robot description, URDF)
Before this commit: robot patrol_robot, 6 links, 5 joints
Links:
- added link camera_optical_link
Joints:
- added joint camera_optical_joint: type fixed, parent camera_link, child camera_optical_link, origin xyz=0 0 0 rpy=-1.57079632679 0 -1.57079632679
- joint ultrasonic_joint: origin xyz=0.23 0 0.00 rpy=0 0 0 -> xyz=0.23 0 0.03 rpy=0 0 0
